File: Hardware/STM32-CSK-Module.sch (KiCad schematic (older format))
At the start: 29 parts, among them J1 Conn_Cortex-JTAG-10, U1 STM32F417VGT, U2 S34ML02G104T, X1 8MHz, X2 32.768kHz

Commit message: Began routing without external flash
Parts:
- removed C18, C19: 0.1uF, Capacitors:CAPC1608N, symbol Capacitor
- removed U2: S34ML02G104T, SOP:SOP50P2000-48N, symbol S34ML02G104T
- X1: footprint (none) -> Clocks:Crystal_Abracon-ABM3
- X2: footprint (none) -> Clocks:Crystal_Abracon-ABS06
Connections:
- net AN0: now reaches U1.35 (PB0)
- net AN1: now reaches U1.36 (PB1)
- net AN2: now reaches U1.15 (PC0)
- net AN3: now reaches U1.16 (PC1)
- net AN4: now reaches U1.17 (PC2)
- net AN5: now reaches U1.18 (PC3)
- net AN6: now reaches U1.33 (PC4)
- net AN7: now reaches U1.34 (PC5)

Commit message: Progress on routing flexible GPIOs
About 50%
Connections:
- net AN0: now also H1.28 (IO34)
- net AN1: now also H1.26 (IO35)
- net AN2: now also H1.18 (IO39)
- net AN3: now also H1.20 (IO38)
- net AN4: now also H1.22 (IO37)
- net AN5: now also H1.24 (IO36)
- net AN6: now also H1.32 (IO32)
- net AN7: now also H1.30 (IO33)
- net IO40: now reaches U1.63 (PC6)
- net IO40: now also H1.16 (IO40)
- net IO41: now reaches U1.64 (PC7)
- net IO41: now also H1.14 (IO41)
- net IO42: now reaches U1.65 (PC8)
- net IO42: now also H1.12 (IO42)
- net IO43: now reaches U1.78 (PC10)
- net IO43: now also H1.10 (IO43)
- net IO44: now reaches U1.79 (PC11)
- net IO44: now also H1.8 (IO44)
- net IO45: now reaches U1.80 (PC12)
- net IO45: now also H1.6 (IO45)
- net IO46: now reaches U1.83 (PD2)
- net IO46: now also H1.4 (IO46)
- net IO47: now reaches U1.84 (PD3)
- net IO47: now also H1.2 (IO47)
- net IO19: now reaches U1.1 (PE2)
- net IO19: now also H1.9 (IO19)
- net IO18: now reaches U1.2 (PE3)
- net IO18: now also H1.11 (IO18)
- net IO17: now reaches U1.3 (PE4)
- net IO17: now also H1.13 (IO17)
- net IO16: now reaches U1.4 (PE5)
- net IO16: now also H1.15 (IO16)

Commit message: Done. Moderately clean.
All used pins routed.
Connections:
- net IO28: now reaches U1.29 (PA4)
- net IO28: now also H1.40 (IO28)
- net IO29: now reaches U1.30 (PA5)
- net IO29: now also H1.38 (IO29)
- net IO30: now reaches U1.31 (PA6)
- net IO30: now also H1.36 (IO30)
- net IO31: now reaches U1.32 (PA7)
- net IO31: now also H1.34 (IO31)
- net IO27: now reaches U1.68 (PA9)
- net IO27: now also H1.42 (IO27)
- net IO26: now reaches U1.69 (PA10)
- net IO26: now also H1.44 (IO26)
- net IO24: now reaches U1.97 (PE0)
- net IO24: now also H1.48 (IO24)
- net IO25: now reaches U1.98 (PE1)
- net IO25: now also H1.46 (IO25)

Commit message: FUCK FUCKING FUCK FUCK FUCK FUCK FUCKING FUCK FUCK
COCK
Parts:
- H1: footprint Connectors:Conn_Samtec-LSS-150 -> (none)
Changed lines of the file:
@@
-$EndComp
-$Comp
-L Conn_Cubesat-PPM H1
-U 1 1 5498CF09
-P 9100 4600
-F 0 "H1" H 9100 5900 60  0000 C CNN
-F 1 "Conn_Cubesat-PPM" H 9100 3300 60  0000 C CNN
-F 2 "Connectors:Conn_Samtec-LSS-150" H 9100 4600 60  0001 C CNN
-F 3 "" H 9100 4600 60  0000 C CNN
-	1    9100 4600
-	1    0    0    -1
-$EndComp
-$Comp
-L Conn_Cubesat-PPM H1
-U 2 1 5498CF75
-P 11700 4600
-F 0 "H1" H 11700 5900 60  0000 C CNN
-F 1 "Conn_Cubesat-PPM" H 11700 3300 60  0000 C CNN
-F 2 "Connectors:Conn_Samtec-LSS-150" H 11700 4600 60  0001 C CNN
-F 3 "" H 11700 4600 60  0000 C CNN
-	2    11700 4600
-	1    0    0    -1
 $EndComp
 $Comp
@@
 Text Label 7600 6900 0    60   ~ 0
 IO25
+$Comp
+L Conn_Cubesat-PPM H1
+U 1 1 54F63AF6
+P 9100 4600
+F 0 "H1" H 9100 5900 60  0000 C CNN
+F 1 "Conn_Cubesat-PPM" H 9100 3300 60  0000 C CNN
+F 2 "" H 9100 4600 60  0000 C CNN
+F 3 "" H 9100 4600 60  0000 C CNN
+	1    9100 4600
+	1    0    0    -1
+$EndComp
+$Comp
+L Conn_Cubesat-PPM H1
+U 2 1 54F63B1B
+P 11700 4600
+F 0 "H1" H 11700 5900 60  0000 C CNN
+F 1 "Conn_Cubesat-PPM" H 11700 3300 60  0000 C CNN
+F 2 "" H 11700 4600 60  0000 C CNN
+F 3 "" H 11700 4600 60  0000 C CNN
+	2    11700 4600
+	1    0    0    -1
+$EndComp
 $EndSCHEMATC
